File: ttaelgam.kicad_pcb (KiCad board)
At the start: 2 copper layers, 212 parts, among them J1 USB_C_Receptacle_USB2.0_16P, J2 Conn_01x04, J3 Conn_01x05, U1 XC6206PxxxMR, U2 RP2040, U3 SRV05-4, U4 W25Q128JVS, Y1 Crystal_GND24

Commit message: 0804over
Parts:
- added S30: MX_stab, marbastlib-mx:STAB_MX_2u, F.Cu at (389.7, 135.0)
- added S63: MX_stab, marbastlib-mx:STAB_MX_2.25u, F.Cu at (394.7, 172.9)
- added S64: MX_stab, marbastlib-mx:STAB_MX_2.25u, F.Cu at (121.1, 199.7)
- added S76: MX_stab, marbastlib-mx:STAB_MX_2.75u, F.Cu at (393.6, 192.5)
- added S81: MX_stab, marbastlib-mx:STAB_MX_2.75u, F.Cu at (192.3, 233.0)
- added S82: MX_stab, marbastlib-mx:STAB_MX_3u, F.Cu at (296.7, 230.7)
- MX34, MX47: footprint marbastlib-mx:SW_MX_HS_CPG151101S11_1u -> marbastlib-mx:SW_MX_HS_CPG151101S11_1.5u
- MX51: footprint marbastlib-mx:SW_MX_HS_CPG151101S11_1u -> marbastlib-mx:SW_MX_HS_CPG151101S11_1.75u_STP_1.25
- MX78, MX79, MX80, MX83: footprint marbastlib-mx:SW_MX_HS_CPG151101S11_1u -> marbastlib-mx:SW_MX_HS_CPG151101S11_1.25u
- moved D42 89.3 mm to (302.3, 176.2), turned to -169 degrees
- moved D58 89.3 mm to (291.9, 197.7), turned to -169 degrees
- moved D74 89.3 mm to (342.3, 207.3), turned to -169 degrees
- moved D10 89.3 mm to (339.9, 120.4), turned to -169 degrees
- moved D12 89.3 mm to (377.3, 113.1), turned to -169 degrees
- moved D29 89.3 mm to (364.1, 144.8), turned to -169 degrees
- moved D44 89.3 mm to (339.7, 169.0), turned to -169 degrees
- moved D45 89.3 mm to (358.4, 165.3), turned to -169 degrees
- moved D46 89.3 mm to (377.1, 161.7), turned to -169 degrees
- moved D59 89.3 mm to (310.6, 194.0), turned to -169 degrees
- moved D61 89.3 mm to (348.0, 186.7), turned to -169 degrees
- moved D62 89.3 mm to (366.7, 183.1), turned to -169 degrees
- moved D63 89.3 mm to (397.1, 177.2), turned to -169 degrees
- moved D72 89.3 mm to (304.9, 214.5), turned to -169 degrees
- moved D73 89.3 mm to (323.6, 210.9), turned to -169 degrees
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